File: IoT Sensor Board/IoTSensorSchematic.sch (EAGLE design)
At the start: 15 parts, among them U1 9DoF IMU, U2 3.3V

Commit message: Schematic completed
I had to change the MPU part, the sparkfun version had a chip that wouldn't play nice on the PCB
Parts:
- removed U1: 9DoF IMU, SparkFun-Sensors:MPU-9250
- added AUXI2C: (no value), pinhead:PINHD-1X2
- added C3, C4: 0.1uF, rcl:C-EUC0805
- added GPIO: (no value), pinhead:PINHD-1X5
- added H1, H2, H3, H4: MOUNT-HOLE3.0, holes:MOUNT-HOLE3.0
- added R10, R7, R8, R9: 10k, rcl:R-EU_R0805
- added R5, R6: 4.7k, rcl:R-EU_R0805
- added S1, S2: (no value), SparkFun-Switches:MOMENTARY-SWITCH-SPST-2-SMD-5.2MM
- added SJ1: (no value), jumper:SJ2W
- added U$1: SMTU_2450N, CustomIoTLibrary:SMTU_2450N
- added U$2: MPU-9250, invensense:MPU-9250
- D1, D2: value (none) -> 1n4148
Connections:
- new net AUX_CL: AUXI2C.1, U$2.AUX_CL
- new net AUX_DATA: AUXI2C.2, U$2.AUX_DA
- new net CS: R10.1, U$2.NCS
- new net N$4: R5.2, SJ1.3
- new net N$5: C3.2, U$2.REGOUT
- new net N$6: R6.2, SJ1.1
- net 3.3V: now also C4.1, R10.2, R7.2, R9.2, SJ1.2, U$2.VDD, U$2.VDDIO
- net ADC: now also GPIO.1
- net GND: now also C3.1, C4.2, R8.1, S1.3, S1.4, S2.3, S2.4, U$1.P$1N, U$2.ADO/SDO, U$2.FSYNC, U$2.GND
- net GPIO0: now also R9.1, S2.1, S2.2
- net GPIO12: now also GPIO.4
- net GPIO13: now also GPIO.5, U$2.INT
- net GPIO14: now also GPIO.3
- net GPIO15: now also R8.2
- net GPIO16: now also GPIO.2
- net GPIO2: now also R7.1
- net GPIO4: now also R6.1, U$2.SDA/SDI
- net GPIO5: now also R5.1, U$2.SCL/SCLK
- net RESET: now also S1.1, S1.2
- net VBAT: now also U$1.P$2P
Other:
- moved on the sheet: C2, R4
