File: IoT Sensor Board/IoTSensorBoardREV2.brd (EAGLE design)
At the start: 40.6 x 44.1 mm, 29 parts, among them Q1 BCW32SMD, Q2 BCW32SMD, U2 3.3V

Commit message: Updated REV2
Silkscreen improved
Parts:
- GPIO: device pinhead:1X04 -> pinhead:1X06
- moved LED1 4.58 mm to (33.0, 19.1)
- moved GPIO 1.80 mm to (38.1, 27.9)
- moved AUXI2C 1.27 mm to (38.1, 15.2)
- renumbered U$2 to U3, U2 to AP2112, X1 to ESP-12
Connections:
- net 3.3V: now also GPIO.5
- net GND: now also GPIO.6
Routing:
- net 3.3V: track 76.9 -> 112.9 mm, vias 4 -> 5
- net GPIO5: track 13.3 -> 20.4 mm, vias 0 -> 2
- net GPIO4: track 13.9 -> 18.9 mm, vias 0 -> 2
- net GPIO16: track 33.1 -> 37.7 mm, vias 1 -> 2
- net ADC: track 39.6 -> 43.5 mm
- net N$3: track 8.56 -> 6.07 mm
- net AUX_DATA: track 24.8 -> 26.0 mm
- net AUX_CL: track 20.5 -> 21.8 mm
Other:
- board text added: "3V3"
- board text added: "ADC"
- board text added: "AUX_CL"
- board text added: "AUX_D"
- board text added: "GND"
- board text added: "GPIO16"
- board text added: "GPIO4"
- board text added: "GPIO5"
- board text added: "RESET"
- board text added: "Vin"
